File: Hardware/duobackpane.sch (EAGLE design)
At the start: 25 parts, among them J1 RJ45-8PTH, U1 BAXXDD0XX

Commit message: Fixed a few bits,
Commit
Parts:
- C1: value (none) -> 33uF
- C2, C3, C4, C5: value (none) -> 100nF
Changed lines of the file:
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@@
 <part name="U1" library="rohm-semi" deviceset="BAXXDD0XX" device=""/>
 <part name="SUPPLY1" library="supply2" deviceset="GND" device=""/>
-<part name="C1" library="resistor" deviceset="CPOL-EU" device="SMCA"/>
-<part name="C2" library="resistor" deviceset="C-EU" device="C0805"/>
-<part name="C3" library="resistor" deviceset="C-EU" device="C0805"/>
-<part name="C4" library="resistor" deviceset="C-EU" device="C0805"/>
-<part name="C5" library="resistor" deviceset="C-EU" device="C0805"/>
+<part name="C1" library="resistor" deviceset="CPOL-EU" device="SMCA" value="33uF"/>
+<part name="C2" library="resistor" deviceset="C-EU" device="C0805" value="100nF"/>
+<part name="C3" library="resistor" deviceset="C-EU" device="C0805" value="100nF"/>
+<part name="C4" library="resistor" deviceset="C-EU" device="C0805" value="100nF"/>
+<part name="C5" library="resistor" deviceset="C-EU" device="C0805" value="100nF"/>
 <part name="LED1" library="led" deviceset="LED" device="SML1206" value="LNK"/>
 <part name="LED2" library="led" deviceset="LED" device="SML1206" value="SPD"/>
